Commit message: fanuc arm in gazebo

File: moveit_resources/fanuc_description/urdf/fanuc.urdf (robot description, URDF)
Before this commit: robot fanuc, 9 links, 8 joints
Links:
- added link dummy_root
- link base_link: mass None -> 10.0
- link link_1: mass None -> 5.0
- link link_2: mass None -> 5.0
- link link_3: mass None -> 5.0
- link link_4: mass None -> 5.0
- link link_5: mass None -> 5.0
- link link_6: mass None -> 3.0
Joints:
- added joint dummy_to_base: type fixed, parent dummy_root, child base_link, origin xyz=0 0 0.1 rpy=0 0 0
